Commit message: Save changes done by Claude to make this compatible with ROS2

File: lwr_description/model/kuka_lwr.gazebo.xacro (robot description, xacro)
@@ -1,8 +1,18 @@
 <?xml version="1.0"?>
 <robot xmlns:xacro="http://www.ros.org/wiki/xacro">
-	<xacro:macro name="kuka_lwr_gazebo" params="name">
+	<!-- controllers_file is the absolute path of the controller manager parameters (controllers.yaml) -->
+	<xacro:macro name="kuka_lwr_gazebo" params="name controllers_file:=''">
+		<!-- the gazebo_ros2_control plugin runs the controller manager in the /${name} namespace
+		     and loads the lwr_hw/LWRHWGazebo hardware interface declared in the ros2_control tag -->
 		<gazebo>
-			<plugin name="${name}_lwr_hw_sim" filename="liblwr_hw_gazebo_plugin.so">
-				<robotNamespace>${name}</robotNamespace>
+			<plugin name="${name}_lwr_hw_sim" filename="libgazebo_ros2_control.so">
+				<ros>
+					<namespace>/${name}</namespace>
+				</ros>
+				<robot_param>robot_description</robot_param>
+				<robot_param_node>/robot_state_publisher</robot_param_node>
+				<xacro:if value="${controllers_file != ''}">
+					<parameters>${controllers_file}</parameters>
+				</xacro:if>
 			</plugin>
 		</gazebo>

File: lwr_description/model/kuka_lwr.urdf.xacro (robot description, xacro)
@@ -5,7 +5,7 @@
 	<xacro:include filename="$(find lwr_description)/model/kuka_materials.xacro"
 	/>
-	<!-- gazebo and transmission models /-->
+	<!-- gazebo and ros2_control models /-->
 	<xacro:include filename="$(find lwr_description)/model/kuka_lwr.gazebo.xacro"/>
-	<xacro:include filename="$(find lwr_description)/model/kuka_lwr.transmission.xacro"/>
+	<xacro:include filename="$(find lwr_description)/model/kuka_lwr.ros2_control.xacro"/>
 	<!-- properties /-->
 	<xacro:property name="base_mass" value="2.0"/>
@@ -19,5 +19,7 @@
 	<xacro:property name="rate_stiffness" value="20000"/> <!-- reflex to stiffness -->
 	<!-- URDF model /-->
-	<xacro:macro name="kuka_lwr" params="parent name *origin">
+	<!-- hardware_interface is gazebo, fri, fril or mock (see kuka_lwr.ros2_control.xacro) /-->
+	<!-- controllers_file is the controller manager parameters file, only used by the gazebo_ros2_control plugin /-->
+	<xacro:macro name="kuka_lwr" params="parent name *origin hardware_interface:=gazebo controllers_file:='' port:=49939 ip:=192.168.0.10 init_file:=''">
 		<!-- First (shoulder) element of the arm. Fixed to its parent. -->
 		<joint name="${parent}_${name}_base_joint" type="fixed">
@@ -31,5 +33,5 @@
 				<mass value="${base_mass}"/>
 				<origin xyz="0 0 0.055"  />
-				<cylinder_inertia_def radius="0.06" length="0.11" mass="${base_mass}"/>
+				<xacro:cylinder_inertia_def radius="0.06" length="0.11" mass="${base_mass}"/>
 			</inertial>
 			<visual>
@@ -68,5 +70,5 @@
 				<mass value="${link_mass}"/>
 				<origin rpy="0 0 0" xyz="0 -0.06 0.130"/>
-				<cuboid_inertia_def length="0.12" width="0.06" height="0.260" mass="${link_mass}"/>
+				<xacro:cuboid_inertia_def length="0.12" width="0.06" height="0.260" mass="${link_mass}"/>
 			</inertial>
 			<visual>
@@ -117,5 +119,5 @@
 				<mass value="${link_mass}"/>
 				<origin rpy="0 0 0" xyz="0 0.06 ${0.130 - 0.06}"/>
-				<cuboid_inertia_def length="0.12" width="0.06" height="0.260" mass="${link_mass}"/>
+				<xacro:cuboid_inertia_def length="0.12" width="0.06" height="0.260" mass="${link_mass}"/>
 			</inertial>
 			<visual>
@@ -166,5 +168,5 @@
 				<mass value="${link_mass}"/>
 				<origin rpy="0 0 0" xyz="0 0.06 0.130"/>
-				<cuboid_inertia_def length="0.12" width="0.06" height="0.260" mass="${link_mass}"/>
+				<xacro:cuboid_inertia_def length="0.12" width="0.06" height="0.260" mass="${link_mass}"/>
 			</inertial>
 			<visual>
@@ -215,5 +217,5 @@
 				<mass value="${link_mass}"/>
 				<origin rpy="0 0 0" xyz="0 -0.06 ${0.130 - 0.06}"/>
-				<cuboid_inertia_def length="0.12" width="0.06" height="0.2600" mass="${link_mass}"/>
+				<xacro:cuboid_inertia_def length="0.12" width="0.06" height="0.2600" mass="${link_mass}"/>
 			</inertial>
 			<visual>
@@ -264,5 +266,5 @@
 				<mass value="${link_mass}"/>
 				<origin rpy="0 0 0" xyz="0 0 0.124"/>
-				<cuboid_inertia_def length="0.12" width="0.06" height="0.248" mass="${link_mass}"/>
+				<xacro:cuboid_inertia_def length="0.12" width="0.06" height="0.248" mass="${link_mass}"/>
 			</inertial>
 			<visual>
@@ -313,5 +315,5 @@
 				<mass value="${wrist_mass}"/>
 				<origin rpy="0 0 0" xyz="0 0 0.0625"/>
-				<cuboid_inertia_def length="0.125" width="0.125" height="0.125" mass="${wrist_mass}"/>
+				<xacro:cuboid_inertia_def length="0.125" width="0.125" height="0.125" mass="${wrist_mass}"/>
 			</inertial>
 			<visual>
@@ -350,5 +352,5 @@
 				<mass value="${tip_mass}"/>
 				<origin xyz="0 0 0"/>
-				<cuboid_inertia_def length="0.1" width="0.1" height="0.1" mass="${tip_mass}"/>
+				<xacro:cuboid_inertia_def length="0.1" width="0.1" height="0.1" mass="${tip_mass}"/>
 			</inertial>
 			<visual>
@@ -366,6 +368,8 @@
 			</collision>
 		</link>
-		<xacro:kuka_lwr_gazebo name="${name}"/>
-		<xacro:kuka_lwr_transmission name="${name}"/>
+		<xacro:if value="${hardware_interface == 'gazebo'}">
+			<xacro:kuka_lwr_gazebo name="${name}" controllers_file="${controllers_file}"/>
+		</xacro:if>
+		<xacro:kuka_lwr_ros2_control name="${name}" hardware_interface="${hardware_interface}" port="${port}" ip="${ip}" init_file="${init_file}"/>
 	</xacro:macro>
 </robot>

File: single_lwr_example/single_lwr_robot/robot/single_lwr_robot.urdf.xacro (robot description, xacro)
@@ -1,35 +1,19 @@
 <?xml version="1.0"?>
 <robot xmlns:xacro="http://www.ros.org/wiki/xacro" name="single_lwr_robot">
+	<!-- arguments, which hardware interface to use (gazebo, fri, fril or mock) and its settings -->
+	<xacro:arg name="hardware_interface" default="gazebo"/>
+	<xacro:arg name="controllers_file" default="$(find single_lwr_robot)/config/controllers.yaml"/>
+	<xacro:arg name="port" default="49939"/>
+	<xacro:arg name="ip" default="192.168.0.10"/>
+	<xacro:arg name="init_file" default="$(find single_lwr_robot)/config/980241-FRI-Driver.init"/>
 	<!-- Include all models -->
 	<xacro:include filename="$(find lwr_description)/model/kuka_lwr.urdf.xacro"/>
-	<!-- and assemble your robot -->
-	<link name="box">
-		<inertial>
-			<mass value="5.0"/>
-			<origin rpy="0 0 0" xyz="0 0 0"/>
-			<inertia ixx="0.01"
-             iyy="0.01"
-             izz="0.01"
-             ixy="0" iyz="0" ixz="0"/>
-		</inertial>
-		<visual>
-			<origin xyz="0 0 0.50" rpy="0 0 0"/>
-			<geometry>
-				<box size="1.0 1.0 1.0"/>
-			</geometry>
-		</visual>
-		<collision>
-			<origin xyz="0 0 0.50" rpy="0 0 0"/>
-			<geometry>
-				<box size="1.0 1.0 1.0"/>
-			</geometry>
-		</collision>
-	</link>
-	<gazebo reference="box">
-		<static>true</static>>
-	</gazebo>
+	<!-- and assemble your robot, the arm is fixed to the world (gazebo welds the "world" link to the ground) -->
+	<link name="world"/>
 	<!-- using the models -->
-	<xacro:kuka_lwr parent="box" name="lwr">
-		<origin xyz="0 0 1" rpy="0 0 0"/>
+	<!-- the name MUST match the name used in the controllers configuration (lwr_a1_joint, ...) -->
+	<xacro:kuka_lwr parent="world" name="lwr" hardware_interface="$(arg hardware_interface)" controllers_file="$(arg controllers_file)"
+	                port="$(arg port)" ip="$(arg ip)" init_file="$(arg init_file)">
+		<origin xyz="0 0 0" rpy="0 0 0"/>
 	</xacro:kuka_lwr>
 </robot>

Commit message: Added cylinder tool at link7 to recreate robot used at Sapienza Univ

File: lwr_description/model/kuka_lwr.gazebo.xacro (robot description, xacro)
@@ -49,4 +49,8 @@
 			<material>Gazebo/Grey</material>
 		</gazebo>
+		<gazebo reference="${name}_tool_link">
+			<gravity>true</gravity>
+			<material>Gazebo/Grey</material>
+		</gazebo>
 	</xacro:macro>
 </robot>

File: lwr_description/model/kuka_lwr.urdf.xacro (robot description, xacro)
@@ -13,6 +13,8 @@
     <xacro:property name="wrist_mass" value="1.1"/>
     <xacro:property name="tip_mass" value="0.25"/>
+	<xacro:property name="tool_mass" value="0.5"/>	<!-- set very arbitrarily /-->
 	<xacro:property name="velocity_scale" value="1"/>
 	<xacro:property name="effort_scale" value="1"/>
+	<xacro:property name="tool_length" value="0.1353"/> <!-- set to match result of SNS paper /-->
 	<xacro:property name="max_stiffness" value="5000"/>
 	<xacro:property name="min_stiffness" value="0"/>
@@ -368,4 +370,30 @@
 			</collision>
 		</link>
+		<!-- Tool: Stick mounted on the flange. The tool frame is at its tip. -->
+		<joint name="${name}_tool_joint" type="fixed">
+			<origin xyz="0 0 ${tool_length}" rpy="0 0 0"/>
+			<parent link="${name}_7_link"/>
+			<child link="${name}_tool_link"/>
+		</joint>
+		<link name="${name}_tool_link">
+			<inertial>
+				<mass value="${tool_mass}"/>
+				<origin xyz="0 0 0.05"/>
+				<xacro:cuboid_inertia_def length="0.02" width="0.02" height="${tool_length}" mass="${tool_mass}"/>
+			</inertial>
+			<visual>
+				<origin xyz="0 0 ${-tool_length/2}" rpy="0 0 0"/>
+				<geometry>
+					<cylinder radius="0.01" length="${tool_length}"/>
+				</geometry>
+			<material name="Kuka/DarkGrey"/>
+			</visual>
+			<collision>
+			<origin xyz="0 0 ${-tool_length/2}" rpy="0 0 0"/>
+			<geometry>
+				<cylinder radius="0.01" length="${tool_length}"/>
+			</geometry>
+			</collision>
+		</link>
 		<xacro:if value="${hardware_interface == 'gazebo'}">
 			<xacro:kuka_lwr_gazebo name="${name}" controllers_file="${controllers_file}"/>

File: single_lwr_example/single_lwr_robot/robot/single_lwr_robot.urdf.xacro (robot description, xacro)
@@ -15,5 +15,5 @@
 	<xacro:kuka_lwr parent="world" name="lwr" hardware_interface="$(arg hardware_interface)" controllers_file="$(arg controllers_file)"
 	                port="$(arg port)" ip="$(arg ip)" init_file="$(arg init_file)">
-		<origin xyz="0 0 0" rpy="0 0 0"/>
+		<origin xyz="0 0 0.0125" rpy="0 0 0"/>	<!-- set to match result of SNS paper /-->
 	</xacro:kuka_lwr>
 </robot>
